Commit message: local: preserve current modified working version

File: resources/robots/b2z1/b2z1.urdf (robot description, URDF)
Before this commit: robot b2_description, 47 links, 46 joints
Links:
- link FL_calf: geometry collision box size=0.05 0.028 0.035; collision box size=0.1 0.0245 0.018
- link FL_hip: geometry visual mesh filename=meshes/FL_hip.dae
- link FL_thigh: geometry collision box size=0.25 0.028 0.04; visual mesh filename=meshes/FL_thigh.dae
- link FR_calf: geometry collision box size=0.05 0.028 0.035; collision box size=0.1 0.0245 0.018
- link FR_hip: geometry visual mesh filename=meshes/FR_hip.dae
- link FR_thigh: geometry collision box size=0.25 0.028 0.04; visual mesh filename=meshes/FR_thigh.dae
- link RL_calf: geometry collision box size=0.05 0.028 0.035; collision box size=0.1 0.0245 0.018
- link RL_hip: geometry visual mesh filename=meshes/RL_hip.dae
- link RL_thigh: geometry collision box size=0.25 0.028 0.04; visual mesh filename=meshes/RL_thigh.dae
- link RR_calf: geometry collision box size=0.05 0.028 0.035; collision box size=0.1 0.0245 0.018
- link RR_hip: geometry visual mesh filename=meshes/RR_hip.dae
- link RR_thigh: geometry collision box size=0.25 0.028 0.04; visual mesh filename=meshes/RR_thigh.dae
- link base_link: geometry collision box size=0.5 0.28 0.15; visual mesh filename=meshes/base_link.dae
- link gripperMover: geometry visual mesh filename=meshes/z1_GripperMover.dae scale=1 1 1
- link gripperStator: geometry visual mesh filename=meshes/z1_GripperStator.dae scale=1 1 1
- link link00: geometry visual mesh filename=meshes/z1_Link00.dae scale=1 1 1
- link link01: geometry visual mesh filename=meshes/z1_Link01.dae scale=1 1 1
- link link02: geometry collision cylinder length=0.051 radius=0.0325; collision cylinder length=0.102 radius=0.0325
- link link03: geometry collision cylinder length=0.059 radius=0.0325; collision cylinder length=0.116 radius=0.02
- link link04: geometry visual mesh filename=meshes/z1_Link04.dae scale=1 1 1
- link link05: geometry visual mesh filename=meshes/z1_Link05.dae scale=1 1 1
- link link06: geometry collision cylinder length=0.051 radius=0.0325; visual mesh filename=meshes/z1_Link06.dae scale=1 1 1
